File: hardware/ctrlSENSE32-C/ctrlSENSE32-C.kicad_sch (KiCad schematic)
At the start: 43 parts, among them J1 USB_C_Receptacle_USB2.0, J2 Screw_Terminal_01x05, J3 PINHD_1x8_Male, J4 PINHD_1x8_Male, U3 TPS54202DDCR, U4 SY8089AAAC, U5 ESP32-C6-MINI-1/U

Commit message: update_test
Parts:
- removed D9: LESD5D5.0CT1G, ctrl_D:SOD-523, symbol ctrl_D:LESD5D5.0CT1G
- added C12, C4: 100nF, ctrl_lib:C_0402, symbol ctrl_lib:C
- added D1: SK6812-EC20, ctrl_D:SMD,2x2mm, symbol ctrl_D:SK6812-EC20
- added D2: 1N5819WS, ctrl_D:SOD-323, symbol ctrl_D:1N5819WS
- added D3: 1N4148W-7-F, ctrl_D:SOD-123, symbol ctrl_D:1N4148W-7-F
- added D9: PSM712-LF-T7, ctrl_D:SOT-23, symbol ctrl_D:PSM712-LF-T7
- added F2, F3: 1206L005/60NR, ctrl_R:R_1206, symbol ctrl_F:F_1206L005/60NR
- added J5: RELAY, ctrl_CON:PV02-3,5-H-P, symbol ctrl_CON:PV2-3,5
- added Q1: MMBT2222ALT1G, ctrl_T:SOT-23, symbol ctrl_T:MMBT2222ALT1G
- added R12, R2, R3, R6, R7: 10k, ctrl_lib:R_0603, symbol ctrl_lib:R
- added R13, R16: 4.7k, ctrl_lib:R_0603, symbol ctrl_lib:R
- added R8: 1k, ctrl_lib:R_0603, symbol ctrl_lib:R
- added SW1: BOOT, ctrl_SW:Omron_B3F-107, symbol ctrl_SW:B3F-1070
- added U1: WS3081, ctrl_U:SOP-8_3.9x4.9mm_P1.27mm, symbol ctrl_U:WS3081
- J3, J4: value PINHD_1x8_Male -> 61300811121; footprint Connector_PinHeader_2.54mm:PinHeader_1x08_P2.54mm_Vertical -> Connector_THT_Wurth:J_Wurth_WR-PHD_61300811121; symbol PCM_SL_Pin_Headers:PINHD_1x8_Male -> Connector_Wurth_WR-PHD:61300811121
Connections:
- net +3.3V: now also Re1.1, C4.1, D3.1, R13.1, R16.1, R2.1, R6.1, U1.8 (VCC)
- net +5V: now also C12.1, D1.1 (VDD), D2.1 (K)
- net +5V_USB: now also D2.2 (A)
- net GND: now also J3.8, C12.2, C4.2, D1.3 (VSS), D9.3 (A), Q1.2 (E), R12.2, R3.2, R7.2, SW1.2 (B), U1.5 (GND)
- net I2C-SCL: now also R13.2
- net I2C-SDA: now also R16.2
- net LED: now also D1.4 (DIN)
- net RS485_A/CAN_L: now also F2.2
- net RS485_B/CAN_H: now also F3.2
- net SPI_CS: now reaches J3.7
- net SPI_CS: now also U5.29 (GPIO23)
- net RS485_DE: now reaches U5.27 (GPIO21)
- net RS485_DE: now also R3.1, U1.2 (~{RE}), U1.3 (DE)
- net RELAY: now reaches U5.28 (GPIO22)
- net RELAY: now also R8.1
- net RS485_RX: now reaches U5.30 (U0RXD/GPIO17)
- net RS485_RX: now also R2.2, U1.1 (RO)
- net RS485_TX: now reaches U5.31 (U0TXD/GPIO16)
- net RS485_TX: now also U1.4 (DI)
- net at Re1.2: now also D3.2, Q1.3 (C)
- net at Re1.5: now also J5.1 (Pin_1)
- net at Re1.6: now also J5.2 (Pin_2)
- net RE/DE: no longer names the net of U5.23 (GPIO9)
- net RE/DE: now also SW1.1 (A)
- new net: Q1.1 (B), R12.1, R8.2
- new net RS485_A: D9.1 (K), F2.1, R6.2, U1.6 (A)
- new net RS485_B: D9.2 (K), F3.1, R7.1, U1.7 (B)
- no-connect marks 6 -> 9
